File: hw/picocart64_v1_lite/picocart64_v1_lite.kicad_sch (KiCad schematic)
At the start: 9 parts, among them J1 Conn_01x04, J2 Conn_01x07, J3 Conn_01x02, J4 Conn_01x01, J5 Conn_01x01, Q1 BSS84, U1 Pico, U4 N64-Cartridge

Commit message: hw: PicoCart64-lite v1.3
Parts:
- added JP1: SolderJumper_2_Open, Jumper:SolderJumper-2_P1.3mm_Open_RoundedPad1.0x1.5mm, symbol Jumper:SolderJumper_2_Open
Connections:
- net +3V3: now also JP1.2 (B)
- net at U1.37 (3V3_EN): now also JP1.1 (A)
- no-connect marks 9 -> 8
Changed lines of the file:
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@@
   (title_block
     (title "PicoCart64-lite")
-    (date "2022-06-29")
-    (rev "V1.2-lite")
+    (date "2022-08-14")
+    (rev "V1.3-lite")
     (company "Konrad Beckmann")
   )
@@
   (junction (at 16.51 78.74) (diameter 0) (color 0 0 0 0)
   )
+  (junction (at 78.74 58.42) (diameter 0) (color 0 0 0 0)
+  )
   (junction (at 91.44 66.04) (diameter 0) (color 0 0 0 0)
   )
@@
   (junction (at 16.51 66.04) (diameter 0) (color 0 0 0 0)
   )
-  (no_connect (at 66.04 55.88))
   (no_connect (at 66.04 60.96))
   (no_connect (at 262.89 83.82))
@@
     (stroke (width 0) (type default) (color 0 0 0 0))
   )
+  (wire (pts (xy 78.74 58.42) (xy 80.01 58.42))
+    (stroke (width 0) (type default) (color 0 0 0 0))
+  )
   (wire (pts (xy 30.48 83.82) (xy 25.4 83.82))
     (stroke (width 0) (type default) (color 0 0 0 0))
@@
     (stroke (width 0) (type default) (color 0 0 0 0))
   )
+  (wire (pts (xy 76.2 55.88) (xy 78.74 55.88))
+    (stroke (width 0) (type default) (color 0 0 0 0))
+  )
   (wire (pts (xy 16.51 66.04) (xy 30.48 66.04))
     (stroke (width 0) (type default) (color 0 0 0 0))
@@
     (stroke (width 0) (type default) (color 0 0 0 0))
   )
-  (wire (pts (xy 66.04 58.42) (xy 71.12 58.42))
+  (wire (pts (xy 66.04 58.42) (xy 78.74 58.42))
     (stroke (width 0) (type default) (color 0 0 0 0))
   )
@@
     (stroke (width 0) (type default) (color 0 0 0 0))
   )
+  (wire (pts (xy 66.04 55.88) (xy 68.58 55.88))
+    (stroke (width 0) (type default) (color 0 0 0 0))
+  )
   (wire (pts (xy 66.04 71.12) (xy 71.12 71.12))
     (stroke (width 0) (type default) (color 0 0 0 0))
   )
   (wire (pts (xy 207.01 35.56) (xy 212.09 35.56))
+    (stroke (width 0) (type default) (color 0 0 0 0))
+  )
+  (wire (pts (xy 78.74 55.88) (xy 78.74 58.42))
     (stroke (width 0) (type default) (color 0 0 0 0))
   )
@@
     )
     (pin "1")
+  )
+  (symbol (lib_id "Jumper:SolderJumper_2_Open") (at 72.39 55.88 0) (unit 1)
+    (in_bom yes) (on_board yes)
+    (property "Reference" "JP1" (id 0) (at 77.47 54.61 0))
+    (property "Value" "SolderJumper_2_Open" (id 1) (at 103.505 55.245 0)
+      (effects (font (size 1.27 1.27)) hide)
+    )
+    (property "Footprint" "Jumper:SolderJumper-2_P1.3mm_Open_RoundedPad1.0x1.5mm" (id 2) (at 72.39 55.88 0)
+      (effects (font (size 1.27 1.27)) hide)
+    )
+    (property "Datasheet" "~" (id 3) (at 72.39 55.88 0)
+      (effects (font (size 1.27 1.27)) hide)
+    )
+    (pin "1")
+    (pin "2")
   )
   (symbol (lib_id "power:+3V3") (at 115.57 148.59 0) (unit 1)
@@
     (pin "1")
   )
-  (symbol (lib_id "power:+3V3") (at 71.12 58.42 270) (unit 1)
-    (in_bom yes) (on_board yes) (fields_autoplaced)
-    (property "Reference" "#PWR0105" (id 0) (at 67.31 58.42 0)
-      (effects (font (size 1.27 1.27)) hide)
-    )
-    (property "Value" "+3V3" (id 1) (at 74.93 58.4199 90)
+  (symbol (lib_id "power:+3V3") (at 80.01 58.42 270) (unit 1)
+    (in_bom yes) (on_board yes) (fields_autoplaced)
+    (property "Reference" "#PWR0105" (id 0) (at 76.2 58.42 0)
+      (effects (font (size 1.27 1.27)) hide)
+    )
+    (property "Value" "+3V3" (id 1) (at 83.82 58.4199 90)
       (effects (font (size 1.27 1.27)) (justify left))
     )
-    (property "Footprint" "" (id 2) (at 71.12 58.42 0)
-      (effects (font (size 1.27 1.27)) hide)
-    )
-    (property "Datasheet" "" (id 3) (at 71.12 58.42 0)
+    (property "Footprint" "" (id 2) (at 80.01 58.42 0)
+      (effects (font (size 1.27 1.27)) hide)
+    )
+    (property "Datasheet" "" (id 3) (at 80.01 58.42 0)
       (effects (font (size 1.27 1.27)) hide)
     )
@@
       (reference "J5") (unit 1) (value "Conn_01x01") (footprint "Connector_PinHeader_2.54mm:PinHeader_1x01_P2.54mm_Vertical")
     )
+    (path "/26be3cc2-c297-45a0-b245-5214add93bfb"
+      (reference "JP1") (unit 1) (value "SolderJumper_2_Open") (footprint "Jumper:SolderJumper-2_P1.3mm_Open_RoundedPad1.0x1.5mm")
+    )
     (path "/4cb68bf6-93e5-4a37-aa35-648d83531bd0"
