File: hw/picocart64_v2/picocart64_v2.kicad_pcb (KiCad board)
At the start: 4 copper layers, 100 x 60 mm, 107 parts, among them J1 USB_C_Receptacle_USB2.0, J2 USB_C_Receptacle_USB2.0, J3 Conn_02x06_Odd_Even, J4 Micro_SD_Card_Det, J5 Conn_01x02, J6 Conn_01x06, Q1 FDN340P, SW1 BootButton, U1 LY68L6400SLIT, U10 USBLC6-2SC6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

Commit message: hw: PicoCart v2: Improve power routing for VBus'
Parts:
- removed kibuzzard-62F96018: G***, kibuzzard-62F96018
- removed kibuzzard-62F964BD: G***, kibuzzard-62F964BD
- added kibuzzard-62F9FC30: G***, kibuzzard-62F9FC30, F.Cu at (184.5, 103.3)
- added kibuzzard-62F9FC40: G***, kibuzzard-62F9FC40, B.Cu at (127.8, 105.3)
